Commit message: Restore calibration services and robot model controllers

File: ffw_description/ros2_control/ffw_sg2_rev1_follower/ffw_sg2_follower.ros2_control.xacro (robot description, xacro)
@@ -609,6 +609,6 @@
         <param name="Return Delay Time">0</param>
         <param name="Profile Velocity">12592</param>
-        <param name="Profile Acceleration Time">500</param>
-        <param name="Profile Time">1000</param>
+        <param name="Profile Acceleration Time">250</param>
+        <param name="Profile Time">500</param>
       </gpio>
       <!-- RIGHT WHEEL -->
@@ -629,6 +629,6 @@
         <param name="Return Delay Time">0</param>
         <param name="Profile Velocity">12592</param>
-        <param name="Profile Acceleration Time">500</param>
-        <param name="Profile Time">1000</param>
+        <param name="Profile Acceleration Time">250</param>
+        <param name="Profile Time">500</param>
       </gpio>
       <!-- REAR WHEEL -->
@@ -649,6 +649,6 @@
         <param name="Return Delay Time">0</param>
         <param name="Profile Velocity">12592</param>
-        <param name="Profile Acceleration Time">500</param>
-        <param name="Profile Time">1000</param>
+        <param name="Profile Acceleration Time">250</param>
+        <param name="Profile Time">500</param>
       </gpio>
     </ros2_control>

File: ffw_description/urdf/common/follower/ffw_follower_body.xacro (robot description, xacro)
@@ -42,5 +42,6 @@
          <origin xyz="0.049483 0 0.102130" rpy="0 0 0" />
          <axis xyz="0 1 0" />
-         <limit velocity="4.8" effort="1000" lower="-0.2317" upper="0.6951" />
+         <!-- <limit velocity="4.8" effort="1000" lower="-0.2317" upper="0.6951" /> -->
+         <limit velocity="4.8" effort="1000" lower="-0.2317" upper="0.83" />
          <dynamics damping="0.1" />
       </joint>

File: ffw_description/urdf/ffw_sg2_rev1_follower/ffw_sg2_follower.urdf (robot description, URDF)
Before this commit: robot ffw_sg2_follower, 50 links, 49 joints
Links:
- link lidar_l_link: mass 0.1 -> None; geometry 
- link lidar_r_link: mass 0.1 -> None; geometry 

File: ffw_description/urdf/ffw_sh5_rev1_follower/ffw_sh5_follower.urdf.xacro (robot description, xacro)
@@ -1,5 +1,5 @@
 <?xml version="1.0"?>
 <robot xmlns:xacro="http://www.ros.org/wiki/xacro" name="ffw_sh5_follower">
-  <xacro:property name="meshes_file_direction" value="package://ffw_description/meshes/$(arg model)" />
+  <xacro:property name="meshes_file_direction" value="package://ffw_description/meshes/common/follower/ffw" />
   <xacro:property name="swerve_meshes_dir" value="package://ffw_description/meshes/common/follower/ffw_swerve" />
   <xacro:arg name="use_sim" default="false" />

Commit message: Revert "Restore calibration services and robot model controllers"
This reverts commit 55f540b66cc844cce63f6c3139c18178b4a2ec7c.

File: ffw_description/ros2_control/ffw_sg2_rev1_follower/ffw_sg2_follower.ros2_control.xacro (robot description, xacro)
@@ -609,6 +609,6 @@
         <param name="Return Delay Time">0</param>
         <param name="Profile Velocity">12592</param>
-        <param name="Profile Acceleration Time">250</param>
-        <param name="Profile Time">500</param>
+        <param name="Profile Acceleration Time">500</param>
+        <param name="Profile Time">1000</param>
       </gpio>
       <!-- RIGHT WHEEL -->
@@ -629,6 +629,6 @@
         <param name="Return Delay Time">0</param>
         <param name="Profile Velocity">12592</param>
-        <param name="Profile Acceleration Time">250</param>
-        <param name="Profile Time">500</param>
+        <param name="Profile Acceleration Time">500</param>
+        <param name="Profile Time">1000</param>
       </gpio>
       <!-- REAR WHEEL -->
@@ -649,6 +649,6 @@
         <param name="Return Delay Time">0</param>
         <param name="Profile Velocity">12592</param>
-        <param name="Profile Acceleration Time">250</param>
-        <param name="Profile Time">500</param>
+        <param name="Profile Acceleration Time">500</param>
+        <param name="Profile Time">1000</param>
       </gpio>
     </ros2_control>

File: ffw_description/urdf/common/follower/ffw_follower_body.xacro (robot description, xacro)
@@ -42,6 +42,5 @@
          <origin xyz="0.049483 0 0.102130" rpy="0 0 0" />
          <axis xyz="0 1 0" />
-         <!-- <limit velocity="4.8" effort="1000" lower="-0.2317" upper="0.6951" /> -->
-         <limit velocity="4.8" effort="1000" lower="-0.2317" upper="0.83" />
+         <limit velocity="4.8" effort="1000" lower="-0.2317" upper="0.6951" />
          <dynamics damping="0.1" />
       </joint>

File: ffw_description/urdf/ffw_sg2_rev1_follower/ffw_sg2_follower.urdf (robot description, URDF)
Before this commit: robot ffw_sg2_follower, 50 links, 49 joints
Links:
- link lidar_l_link: mass None -> 0.1; geometry visual cylinder length=0.03 radius=0.03
- link lidar_r_link: mass None -> 0.1; geometry visual cylinder length=0.03 radius=0.03

File: ffw_description/urdf/ffw_sh5_rev1_follower/ffw_sh5_follower.urdf.xacro (robot description, xacro)
@@ -1,5 +1,5 @@
 <?xml version="1.0"?>
 <robot xmlns:xacro="http://www.ros.org/wiki/xacro" name="ffw_sh5_follower">
-  <xacro:property name="meshes_file_direction" value="package://ffw_description/meshes/common/follower/ffw" />
+  <xacro:property name="meshes_file_direction" value="package://ffw_description/meshes/$(arg model)" />
   <xacro:property name="swerve_meshes_dir" value="package://ffw_description/meshes/common/follower/ffw_swerve" />
   <xacro:arg name="use_sim" default="false" />
