Commit message: fix(runtime): recover current AD source and installed launch configuration
Copy ai_worker_full_real_20261015 source, preserve the four installed launch/config overrides, and record recovery provenance. Keep the pre-sync host snapshot on backup/host-before-ad-sync-20261027.

File: ffw_description/ros2_control/ffw_a3/ffw_a3.ros2_control.xacro (robot description, xacro)
@@ -1,5 +1,5 @@
 <?xml version="1.0"?>
 <robot xmlns:xacro="http://www.ros.org/wiki/xacro">
-  <xacro:macro name="ffw_a3_system" params="use_sim:=^|false use_mock_hardware:=^|false mock_sensor_commands:=^|false">
+  <xacro:macro name="ffw_a3_system" params="use_sim:=^|false use_mock_hardware:=^|false mock_sensor_commands:=^|false port_name:=/dev/serial/by-id/usb-ROBOTIS_Avatar_Controller_315738613434-if00">
     <xacro:property name="initial_positions" value="${load_yaml(initial_positions_file)['initial_positions']}"/>
     <ros2_control name="ffw_a3" type="system" is_async="true">
@@ -18,5 +18,5 @@
           <xacro:unless value="${use_mock_hardware}">
             <plugin>dynamixel_hardware_interface/DynamixelHardware</plugin>
-            <param name="port_name">/dev/serial/by-id/usb-ROBOTIS_Avatar_Controller_315738613434-if00</param>
+            <param name="port_name">${port_name}</param>
             <param name="baud_rate">4000000</param>
             <param name="dynamixel_model_folder">/param/dxl_model</param>

File: ffw_description/ros2_control/ffw_sh5_rev1_follower/ffw_sh5_follower.ros2_control.xacro (robot description, xacro)
@@ -1,4 +1,5 @@
 <?xml version="1.0"?>
 <robot xmlns:xacro="http://www.ros.org/wiki/xacro">
+  <xacro:arg name="sh5_thumb_contact_guard" default="false" />
   <xacro:include filename="$(find ffw_description)/ros2_control/$(arg model)/ffw_sh5_follower.joints.xacro" />
   <xacro:include filename="$(find robotis_hand_description)/ros2_control/hx5_d20_rev2/hx5_d20_left.joints.xacro" />
@@ -26,4 +27,7 @@
             <param name="number_of_transmissions">60</param>
             <param name="disable_torque_at_init">true</param>
+            <!-- Backdrive relief for joint3 on both thumbs preserves ordinary grasp force. -->
+            <param name="sh5_thumb_contact_guard">$(arg sh5_thumb_contact_guard)</param>
+            <param name="enable_hand_recovery">true</param>
             <param name="dynamixel_state_pub_msg_name">ffw_follower/dxl_state</param>
             <param name="get_dynamixel_data_srv_name">ffw_follower/get_dxl_data</param>

File: ffw_description/urdf/ffw_a3/ffw_a3.urdf.xacro (robot description, xacro)
@@ -5,4 +5,5 @@
   <xacro:arg name="mock_sensor_commands" default="false" />
   <xacro:arg name="prefix" default="" />
+  <xacro:arg name="port_name" default="/dev/serial/by-id/usb-ROBOTIS_Avatar_Controller_315738613434-if00" />
   <xacro:include filename="$(find ffw_description)/urdf/common/leader/ffw_mini_leader_body.urdf.xacro" />
   <xacro:include filename="$(find ffw_description)/ros2_control/ffw_a3/ffw_a3.ros2_control.xacro" />
@@ -14,4 +15,5 @@
       use_sim="$(arg use_sim)"
       use_mock_hardware="$(arg use_mock_hardware)"
-      mock_sensor_commands="$(arg mock_sensor_commands)" />
+      mock_sensor_commands="$(arg mock_sensor_commands)"
+      port_name="$(arg port_name)" />
 </robot>
